File: Projects/Client Name/DF_ESC/Design/DF_ESC/DF_ESC_rev01_1/BLOCK DIAGRAM.kicad_sch (KiCad schematic)
At the start: 0 parts

Commit message: libraries & schemtics
Other:
- note added: "+3V3"
- note added: "+5V"
- note added: "0 - +60V"
- note added: "03407610395"
- note added: "Muhammad Moiz"
- note added: "STEP-DOWN 3V3"
- note added: "VDC"
- note added: "moizrai765yt@gmail.com"
- note removed: "V_SUPPLY"
- company: (none) -> coVenture
- title: (none) -> BLOCK DIAGRAM
Changed lines of the file:
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@@
 	(generator_version "8.0")
 	(paper "A4")
-	(polyline
-		(pts
-			(xy 251.46 106.68) (xy 276.86 106.68)
+	(title_block
+		(title "BLOCK DIAGRAM")
+		(rev "rev01_1")
+		(company "coVenture")
+	)
+	(polyline
+		(pts
+			(xy 99.06 81.28) (xy 180.34 81.28)
+		)
+		(stroke
+			(width 2.54)
+			(type solid)
+			(color 132 0 0 1)
+		)
+	)
+	(polyline
+		(pts
+			(xy 250.19 106.68) (xy 275.59 106.68)
 		)
 		(stroke
@@
 	(polyline
 		(pts
+			(xy 162.56 111.76) (xy 194.31 111.76)
+		)
+		(stroke
+			(width 0)
+			(type solid)
+		)
+	)
+	(polyline
+		(pts
 			(xy 34.29 116.84) (xy 34.29 130.81)
 		)
@@
 	(polyline
 		(pts
+			(xy 181.61 106.68) (xy 181.61 111.76)
+		)
+		(stroke
+			(width 1)
+			(type solid)
+			(color 132 0 0 1)
+		)
+	)
+	(polyline
+		(pts
 			(xy 46.99 96.52) (xy 63.5 96.52)
 		)
@@
 	(polyline
 		(pts
-			(xy 246.38 102.87) (xy 250.19 102.87)
+			(xy 208.28 96.52) (xy 208.28 107.95)
+		)
+		(stroke
+			(width 0)
+			(type solid)
+		)
+	)
+	(polyline
+		(pts
+			(xy 223.52 81.28) (xy 223.52 95.25)
 		)
 		(stroke
 			(width 2.54)
 			(type solid)
-		)
-	)
-	(polyline
-		(pts
-			(xy 208.28 96.52) (xy 208.28 107.95)
-		)
-		(stroke
-			(width 0)
-			(type solid)
-		)
-	)
-	(polyline
-		(pts
-			(xy 276.86 106.68) (xy 276.86 96.52)
+			(color 132 0 0 1)
+		)
+	)
+	(polyline
+		(pts
+			(xy 180.34 81.28) (xy 223.52 81.28)
+		)
+		(stroke
+			(width 2.54)
+			(type solid)
+			(color 132 0 0 1)
+		)
+	)
+	(polyline
+		(pts
+			(xy 275.59 106.68) (xy 275.59 96.52)
+		)
+		(stroke
+			(width 0)
+			(type solid)
+		)
+	)
+	(polyline
+		(pts
+			(xy 162.56 111.76) (xy 158.75 111.76)
 		)
 		(stroke
@@
 	(polyline
 		(pts
+			(xy 158.75 111.76) (xy 158.75 125.73)
+		)
+		(stroke
+			(width 0)
+			(type solid)
+		)
+	)
+	(polyline
+		(pts
+			(xy 142.24 120.65) (xy 142.24 115.57)
+		)
+		(stroke
+			(width 1)
+			(type solid)
+			(color 132 0 0 1)
+		)
+	)
+	(polyline
+		(pts
+			(xy 158.75 120.65) (xy 142.24 120.65)
+		)
+		(stroke
+			(width 1)
+			(type solid)
+			(color 132 0 0 1)
+		)
+	)
+	(polyline
+		(pts
 			(xy 43.18 102.87) (xy 67.31 102.87)
 		)
@@
 	(polyline
 		(pts
+			(xy 194.31 125.73) (xy 194.31 111.76)
+		)
+		(stroke
+			(width 0)
+			(type solid)
+		)
+	)
+	(polyline
+		(pts
 			(xy 40.64 134.62) (xy 72.39 134.62)
 		)
@@
 	(polyline
 		(pts
+			(xy 245.11 101.6) (xy 245.11 102.87)
+		)
+		(stroke
+			(width 0)
+			(type solid)
+		)
+	)
+	(polyline
+		(pts
+			(xy 158.75 125.73) (xy 194.31 125.73)
+		)
+		(stroke
+			(width 0)
+			(type solid)
+		)
+	)
+	(polyline
+		(pts
 			(xy 208.28 107.95) (xy 237.49 107.95)
 		)
@@
 	(polyline
 		(pts
+			(xy 245.11 102.87) (xy 248.92 102.87)
+		)
+		(stroke
+			(width 2.54)
+			(type solid)
+			(color 132 0 0 1)
+		)
+	)
+	(polyline
+		(pts
 			(xy 100.33 76.2) (xy 245.11 76.2)
 		)
@@
 			(width 2.54)
 			(type solid)
+			(color 132 0 0 1)
 		)
 	)
@@
 	(polyline
 		(pts
-			(xy 251.46 96.52) (xy 276.86 96.52)
+			(xy 250.19 96.52) (xy 275.59 96.52)
 		)
 		(stroke
@@
 	(polyline
 		(pts
+			(xy 245.11 102.87) (xy 238.76 102.87)
+		)
+		(stroke
+			(width 2.54)
+			(type solid)
+			(color 132 0 0 1)
+		)
+	)
+	(polyline
+		(pts
 			(xy 154.94 96.52) (xy 154.94 106.68)
 		)
@@
 	(polyline
 		(pts
+			(xy 180.34 81.28) (xy 180.34 95.25)
+		)
+		(stroke
+			(width 2.54)
+			(type solid)
+			(color 132 0 0 1)
+		)
+	)
+	(polyline
+		(pts
 			(xy 208.28 96.52) (xy 237.49 96.52)
 		)
@@
 	(polyline
 		(pts
-			(xy 251.46 96.52) (xy 251.46 106.68)
-		)
-		(stroke
-			(width 0)
-			(type solid)
+			(xy 250.19 96.52) (xy 250.19 106.68)
+		)
+		(stroke
+			(width 0)
+			(type solid)
+		)
+	)
+	(text "STEP-DOWN\n3V3"
+		(exclude_from_sim no)
+		(at 176.53 119.38 0)
+		(effects
+			(font
+				(size 3.81 3.81)
+				(thickness 0.762)
+				(bold yes)
+			)
 		)
 	)
@@
 		)
 	)
-	(text "V_SUPPLY"
+	(text "+5V"
+		(exclude_from_sim no)
+		(at 184.15 109.22 0)
+		(effects
+			(font
+				(size 1 1)
+				(thickness 0.762)
+				(bold yes)
+			)
+		)
+	)
+	(text "VDC"
 		(exclude_from_sim no)
 		(at 54.61 81.28 0)
@@
 		)
 	)
+	(text "Muhammad Moiz\n"
+		(exclude_from_sim no)
+		(at 210.566 168.656 0)
+		(effects
+			(font
+				(size 1.27 1.27)
+			)
+		)
+	)
 	(text "USB\n"
 		(exclude_from_sim no)
@@
 		)
 	)
+	(text "moizrai765yt@gmail.com\n"
+		(exclude_from_sim no)
+		(at 214.63 171.704 0)
+		(effects
+			(font
+				(size 1.27 1.27)
+			)
+		)
+	)
 	(text "SERVO"
 		(exclude_from_sim no)
@@
 				(thickness 0.762)
 				(bold yes)
+			)
+		)
+	)
+	(text "03407610395\n"
+		(exclude_from_sim no)
+		(at 209.55 177.8 0)
+		(effects
+			(font
+				(size 1.27 1.27)
 			)
 		)
@@
 		)
 	)
+	(text "+3V3"
+		(exclude_from_sim no)
+		(at 148.59 119.38 0)
+		(effects
+			(font
+				(size 1 1)
+				(thickness 0.762)
+				(bold yes)
+			)
+		)
+	)
 	(text "COM"
 		(exclude_from_sim no)
@@
 	(text "MOTOR"
 		(exclude_from_sim no)
-		(at 262.89 101.6 0)
-		(effects
-			(font
+		(at 261.62 101.6 0)
+		(effects
+			(font
+				(size 3.81 3.81)
+				(thickness 0.762)
+				(bold yes)
+			)
+		)
+	)
+	(text "0 - +60V"
+		(exclude_from_sim no)
+		(at 54.61 73.66 0)
+		(effects
+			(font
