File: Projects/Client Name/DF_ESC/Design/DF_ESC/DF_ESC_rev01_1/OVERVIEW.kicad_sch (KiCad schematic)
At the start: 0 parts

Commit message: libraries & schemtics
Other:
- note added: "USB"
Changed lines of the file:
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@@
 	(generator_version "8.0")
 	(paper "A4")
+	(text "USB"
+		(exclude_from_sim no)
+		(at 138.43 27.94 0)
+		(effects
+			(font
+				(size 10 10)
+				(thickness 2)
+				(bold yes)
+			)
+		)
+	)
 )
