File: Projects/Client Name/DF_ESC/Design/DF_ESC/DF_ESC_rev01_1/FILTERS.kicad_sch (KiCad schematic)
At the start: 0 parts

Commit message: libraries & schemtics
Parts:
- added C43, C45, C47, C49: 4n7, symbol Device:C
- added C44, C46, C48, C50: 100n, symbol Device:C
- added J5: Conn_01x06, symbol Connector_Generic:Conn_01x06
- added R27, R29, R31, R33: 2k2, symbol Device:R
- added R28, R30, R32, R34: 10k, symbol Device:R
Connections:
- new net +3V3: C44.1, C46.1, C48.1, C50.1, R27.1, R29.1, R31.1, R33.1
- new net +5V: J5.6 (Pin_6)
- new net GND: C43.2, C44.2, C45.2, C46.2, C47.2, C48.2, C49.2, C50.2, J5.1 (Pin_1)
- new net HALL_1_IN: C43.1, J5.4 (Pin_4), R27.2, R28.1
- new net HALL_1_OUT: R28.2
- new net HALL_2_IN: C45.1, J5.3 (Pin_3), R29.2, R30.1
- new net HALL_2_OUT: R30.2
- new net HALL_3_IN: C47.1, J5.2 (Pin_2), R31.2, R32.1
- new net HALL_3_OUT: R32.2
- new net TEMP_IN: C49.1, J5.5 (Pin_5), R33.2, R34.1
- new net TEMP_MOTOR: R34.2
Other:
- note added: "03407610395"
- note added: "FILTERS"
- note added: "HALL ENCODER INPUT"
- note added: "HALL ENCODER OUTPUT"
- note added: "HALL_1 FILTER"
- note added: "HALL_2 FILTER"
- note added: "HALL_3 FILTER"
- note added: "Muhammad Moiz"
- note added: "TEMP_MOTOR FILTER"
- note added: "TO MCU =>"
- note added: "moizrai765yt@gmail.com"
- company: (none) -> coVenture
- title: (none) -> FILTERS

Commit message: updated footprints
Parts:
- C43, C44, C45, C46, C47, C48, C49, C50: footprint (none) -> Capacitor_SMD:C_0603_1608Metric
- J5: footprint (none) -> Connector_PinHeader_1.00mm:PinHeader_1x06_P1.00mm_Vertical
- R27, R28, R29, R30, R31, R32, R33, R34: footprint (none) -> Resistor_SMD:R_0201_0603Metric
Changed lines of the file:
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@@
 			)
 		)
-		(property "Footprint" ""
+		(property "Footprint" "Capacitor_SMD:C_0603_1608Metric"
 			(at 139.3952 168.91 0)
 			(effects
@@
 			)
 		)
-		(property "Footprint" ""
+		(property "Footprint" "Resistor_SMD:R_0201_0603Metric"
 			(at 112.522 171.45 90)
 			(effects
@@
 			)
 		)
-		(property "Footprint" ""
+		(property "Footprint" "Capacitor_SMD:C_0603_1608Metric"
 			(at 115.2652 187.96 0)
 			(effects
@@
 			)
 		)
-		(property "Footprint" ""
+		(property "Footprint" "Resistor_SMD:R_0201_0603Metric"
 			(at 128.27 95.758 90)
 			(effects
@@
 			)
 		)
-		(property "Footprint" ""
+		(property "Footprint" "Resistor_SMD:R_0201_0603Metric"
 			(at 112.522 87.63 90)
 			(effects
@@
 			)
 		)
-		(property "Footprint" ""
+		(property "Footprint" "Capacitor_SMD:C_0603_1608Metric"
 			(at 115.2652 62.23 0)
 			(effects
@@
 			)
 		)
-		(property "Footprint" ""
+		(property "Footprint" "Resistor_SMD:R_0201_0603Metric"
 			(at 112.522 45.72 90)
 			(effects
@@
 			)
 		)
-		(property "Footprint" ""
+		(property "Footprint" "Resistor_SMD:R_0201_0603Metric"
 			(at 128.27 179.578 90)
 			(effects
@@
 			)
 		)
-		(property "Footprint" ""
+		(property "Footprint" "Capacitor_SMD:C_0603_1608Metric"
 			(at 115.2652 146.05 0)
 			(effects
@@
 			)
 		)
-		(property "Footprint" ""
+		(property "Footprint" "Resistor_SMD:R_0201_0603Metric"
 			(at 112.522 129.54 90)
 			(effects
@@
 			)
 		)
-		(property "Footprint" ""
+		(property "Footprint" "Capacitor_SMD:C_0603_1608Metric"
 			(at 139.3952 85.09 0)
 			(effects
@@
 			)
 		)
-		(property "Footprint" ""
+		(property "Footprint" "Capacitor_SMD:C_0603_1608Metric"
 			(at 139.3952 127 0)
 			(effects
@@
 			)
 		)
-		(property "Footprint" ""
+		(property "Footprint" "Resistor_SMD:R_0201_0603Metric"
 			(at 128.27 53.848 90)
 			(effects
@@
 			)
 		)
-		(property "Footprint" ""
+		(property "Footprint" "Capacitor_SMD:C_0603_1608Metric"
 			(at 115.2652 104.14 0)
 			(effects
@@
 			)
 		)
-		(property "Footprint" ""
+		(property "Footprint" "Resistor_SMD:R_0201_0603Metric"
 			(at 128.27 137.668 90)
 			(effects
@@
 			)
 		)
-		(property "Footprint" ""
+		(property "Footprint" "Connector_PinHeader_1.00mm:PinHeader_1x06_P1.00mm_Vertical"
 			(at 27.94 74.93 0)
 			(effects
@@
 			)
 		)
-		(property "Footprint" ""
+		(property "Footprint" "Capacitor_SMD:C_0603_1608Metric"
 			(at 139.3952 43.18 0)
 			(effects
