File: Projects/Client Name/DF_ESC/Design/DF_ESC/DF_ESC_rev01_1/MOSFETs.kicad_sch (KiCad schematic)
At the start: 0 parts

Commit message: libraries & schemtics
Parts:
- added C59, C60: 2n2, symbol Device:C
- added HSBA15810C1, HSBA15810C2, HSBA15810C3, HSBA15810C4, HSBA15810C5, HSBA15810C6: ~, symbol HSBA15810C:HSBA15810C
- added J10, J8, J9: Conn_01x01, symbol Connector_Generic:Conn_01x01
- added NT1, NT2, NT3, NT4, NT5, NT6, NT7, NT8: NetTie_2, symbol Device:NetTie_2
- added R39K, R39K1, R39K2, R48, R49, R50, R53, R54, R57, R58, R59: 4R7, symbol Device:R
- added R51, R52, R55, R56: 100R, symbol Device:R
Connections:
- new net +VDC: HSBA15810C1.5 (D), HSBA15810C4.5 (D), HSBA15810C6.5 (D)
- new net GND: NT3.1, NT6.1, NT8.1, R39K.1, R39K1.1, R39K2.1
- new net H1_LOW: HSBA15810C2.1 (S), NT2.2
- new net H1_VS: NT1.1
- new net H2_LOW: HSBA15810C3.1 (S), NT5.2
- new net H2_VS: NT4.1
- new net H3_LOW: HSBA15810C5.1 (S), NT8.2
- new net H3_VS: NT7.1
- new net M_H1: R48.1
- new net M_H1_RG: HSBA15810C1.4 (G), R48.2
- new net M_H2: R53.1
- new net M_H2_RG: HSBA15810C4.4 (G), R53.2
- new net M_H3: R58.1
- new net M_H3_RG: HSBA15810C6.4 (G), R58.2
- new net M_L1: R49.1
- new net M_L1_RG: HSBA15810C2.4 (G), R39K.2, R49.2
- new net M_L2: R54.1
- new net M_L2_RG: HSBA15810C3.4 (G), R39K1.2, R54.2
- new net M_L3: R59.1
- new net M_L3_RG: HSBA15810C5.4 (G), R39K2.2, R59.2
- new net PHASE_1: HSBA15810C1.1 (S), HSBA15810C2.5 (D), J8.1 (Pin_1), NT1.2
- new net PHASE_2: HSBA15810C3.5 (D), HSBA15810C4.1 (S), J9.1 (Pin_1), NT4.2
- new net PHASE_3: HSBA15810C5.5 (D), HSBA15810C6.1 (S), J10.1 (Pin_1), NT7.2
- new net S1_N: C59.1, R51.2
- new net S1_P: C59.2, R52.2
- new net S2_N: C60.1, R55.2
- new net S2_P: C60.2, R56.2
- new net SH1_N: NT2.1, R50.2, R51.1
- new net SH1_P: NT3.2, R50.1, R52.1
- new net SH2_N: NT5.1, R55.1, R57.2
- new net SH2_P: NT6.2, R56.1, R57.1
- no-connect marks 0 -> 36
Other:
- note added: "03407610395"
- note added: "Hx_VS"
- note added: "MCU SENSING FEEDBACK FOR EACH PHASE"
- note added: "MOSFETs"
- note added: "Muhammad Moiz"
- note added: "OUTPUT PHASE 1"
- note added: "OUTPUT PHASE 2"
- note added: "OUTPUT PHASE 3"
- note added: "PHASE 1"
- note added: "PHASE 2"
- note added: "PHASE 3"
- note added: "PLACE AS CLOSE AS POSSIBLE TO THE BULK CAPACITANCE"
- note added: "Q_CONTROL"
- note added: "Q_SOURCES"
- note added: "ROUTE AS KELVING CONNECTIONS"
- note added: "SENSE 1"
- note added: "SENSE 2"
- note added: "moizrai765yt@gmail.com"
- company: (none) -> coVenture
- title: (none) -> MOSFETs

Commit message: updated footprints
Parts:
- C59, C60: footprint (none) -> Capacitor_SMD:C_0603_1608Metric
- HSBA15810C1, HSBA15810C2, HSBA15810C3, HSBA15810C4, HSBA15810C5, HSBA15810C6: footprint (none) -> HSBA15810C:HSBA15810C
- J10, J8, J9: footprint (none) -> Connector_PinHeader_1.00mm:PinHeader_1x01_P1.00mm_Vertical
- NT1, NT2, NT3, NT4, NT5, NT6, NT7, NT8: footprint (none) -> NetTie:NetTie-2_SMD_Pad0.5mm
- R39K1, R39K2, R48, R49, R50, R51, R52, R53, R54, R55, R56, R57, R58, R59: footprint (none) -> Resistor_SMD:R_0201_0603Metric
- R39K3: renamed from R39K; footprint (none) -> Resistor_SMD:R_0201_0603Metric
Changed lines of the file:
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@@
 			)
 		)
-		(property "Footprint" ""
+		(property "Footprint" "NetTie:NetTie-2_SMD_Pad0.5mm"
 			(at 215.9 124.46 0)
 			(effects
@@
 			)
 		)
-		(property "Footprint" ""
+		(property "Footprint" "Connector_PinHeader_1.00mm:PinHeader_1x01_P1.00mm_Vertical"
 			(at 276.86 105.41 0)
 			(effects
@@
 			)
 		)
-		(property "Footprint" ""
+		(property "Footprint" "Connector_PinHeader_1.00mm:PinHeader_1x01_P1.00mm_Vertical"
 			(at 276.86 74.93 0)
 			(effects
@@
 			)
 		)
-		(property "Footprint" ""
+		(property "Footprint" "Resistor_SMD:R_0201_0603Metric"
 			(at 74.93 125.222 90)
 			(effects
@@
 			)
 		)
-		(property "Footprint" ""
+		(property "Footprint" "NetTie:NetTie-2_SMD_Pad0.5mm"
 			(at 97.79 142.24 0)
 			(effects
@@
 			)
 		)
-		(property "Footprint" ""
+		(property "Footprint" "HSBA15810C:HSBA15810C"
 			(at 78.74 114.3 0)
 			(effects
@@
 			)
 		)
-		(property "Footprint" ""
+		(property "Footprint" "Resistor_SMD:R_0201_0603Metric"
 			(at 203.2 62.738 90)
 			(effects
@@
 			)
 		)
-		(property "Footprint" ""
+		(property "Footprint" "Capacitor_SMD:C_0603_1608Metric"
 			(at 61.9252 135.89 0)
 			(effects
@@
 		(on_board yes)
 		(dnp no)
-		(property "Reference" "R39K"
+		(property "Reference" "R39K3"
 			(at 68.58 109.2201 0)
 			(effects
@@
 			)
 		)
-		(property "Footprint" ""
+		(property "Footprint" "Resistor_SMD:R_0201_0603Metric"
 			(at 72.898 107.95 90)
 			(effects
@@
 			(project "DF_ESC_rev01_1"
 				(path "/e63e39d7-6ac0-4ffd-8aa3-1841a4541b55/9a0f3e7c-c741-4f72-a420-b5ade149b6b8"
-					(reference "R39K")
+					(reference "R39K3")
 					(unit 1)
 				)
@@
 			)
 		)
-		(property "Footprint" ""
+		(property "Footprint" "Resistor_SMD:R_0201_0603Metric"
 			(at 74.93 135.382 90)
 			(effects
@@
 			)
 		)
-		(property "Footprint" ""
+		(property "Footprint" "HSBA15810C:HSBA15810C"
 			(at 147.32 114.3 0)
 			(effects
@@
 			)
 		)
-		(property "Footprint" ""
+		(property "Footprint" "Capacitor_SMD:C_0603_1608Metric"
 			(at 130.5052 135.89 0)
 			(effects
@@
 			)
 		)
-		(property "Footprint" ""
+		(property "Footprint" "Connector_PinHeader_1.00mm:PinHeader_1x01_P1.00mm_Vertical"
 			(at 276.86 90.17 0)
 			(effects
@@
 			)
 		)
-		(property "Footprint" ""
+		(property "Footprint" "NetTie:NetTie-2_SMD_Pad0.5mm"
 			(at 208.28 81.28 0)
 			(effects
@@
 			)
 		)
-		(property "Footprint" ""
+		(property "Footprint" "Resistor_SMD:R_0201_0603Metric"
 			(at 133.35 102.108 90)
 			(effects
@@
 			)
 		)
-		(property "Footprint" ""
+		(property "Footprint" "Resistor_SMD:R_0201_0603Metric"
 			(at 64.77 62.738 90)
 			(effects
@@
 			)
 		)
-		(property "Footprint" ""
+		(property "Footprint" "Resistor_SMD:R_0201_0603Metric"
 			(at 133.35 62.738 90)
 			(effects
@@
 			)
 		)
-		(property "Footprint" ""
+		(property "Footprint" "Resistor_SMD:R_0201_0603Metric"
 			(at 168.148 132.08 90)
 			(effects
@@
 			)
 		)
-		(property "Footprint" ""
+		(property "Footprint" "Resistor_SMD:R_0201_0603Metric"
 			(at 141.478 107.95 90)
 			(effects
@@
 			)
 		)
-		(property "Footprint" ""
+		(property "Footprint" "HSBA15810C:HSBA15810C"
 			(at 217.17 114.3 0)
 			(effects
@@
 			)
 		)
-		(property "Footprint" ""
+		(property "Footprint" "Resistor_SMD:R_0201_0603Metric"
 			(at 99.568 132.08 90)
 			(effects
@@
 			)
 		)
-		(property "Footprint" ""
+		(property "Footprint" "Resistor_SMD:R_0201_0603Metric"
 			(at 203.2 102.108 90)
 			(effects
@@
 			)
 		)
-		(property "Footprint" ""
+		(property "Footprint" "Resistor_SMD:R_0201_0603Metric"
 			(at 143.51 125.222 90)
 			(effects
@@
 			)
 		)
-		(property "Footprint" ""
+		(property "Footprint" "NetTie:NetTie-2_SMD_Pad0.5mm"
 			(at 69.85 81.28 0)
 			(effects
@@
 			)
 		)
-		(property "Footprint" ""
+		(property "Footprint" "NetTie:NetTie-2_SMD_Pad0.5mm"
 			(at 166.37 123.19 0)
 			(effects
@@
 			)
 		)
-		(property "Footprint" ""
+		(property "Footprint" "HSBA15810C:HSBA15810C"
 			(at 148.59 74.93 0)
 			(effects
@@
 			)
 		)
-		(property "Footprint" ""
+		(property "Footprint" "Resistor_SMD:R_0201_0603Metric"
 			(at 143.51 135.382 90)
 			(effects
@@
 			)
 		)
-		(property "Footprint" ""
+		(property "Footprint" "NetTie:NetTie-2_SMD_Pad0.5mm"
 			(at 97.79 123.19 0)
 			(effects
@@
 			)
 		)
-		(property "Footprint" ""
+		(property "Footprint" "HSBA15810C:HSBA15810C"
 			(at 80.01 74.93 0)
 			(effects
@@
 			)
 		)
-		(property "Footprint" ""
+		(property "Footprint" "Resistor_SMD:R_0201_0603Metric"
 			(at 64.77 102.108 90)
 			(effects
@@
 			)
 		)
-		(property "Footprint" ""
+		(property "Footprint" "HSBA15810C:HSBA15810C"
 			(at 218.44 74.93 0)
 			(effects
@@
 			)
 		)
-		(property "Footprint" ""
+		(property "Footprint" "Resistor_SMD:R_0201_0603Metric"
 			(at 211.328 107.95 90)
 			(effects
@@
 			)
 		)
-		(property "Footprint" ""
+		(property "Footprint" "NetTie:NetTie-2_SMD_Pad0.5mm"
 			(at 166.37 142.24 0)
 			(effects
@@
 			)
 		)
-		(property "Footprint" ""
+		(property "Footprint" "NetTie:NetTie-2_SMD_Pad0.5mm"
 			(at 138.43 81.28 0)
 			(effects
