File: Projects/Client Name/DF_ESC/Design/DF_ESC/DF_ESC_rev01_1/MCU.kicad_sch (KiCad schematic)
At the start: 0 parts

Commit message: DRV8302
Parts:
- added C1, C11, C12, C15, C16, C2, C3, C4, C5, C6, C8: 100n, symbol Device:C
- added C10, C9: 2u2, symbol Device:C
- added C13, C14: 10p, symbol Device:C
- added C17, C7: 10u, symbol Device:C
- added D1: LED, symbol Device:LED
- added D2: LED_G, symbol Device:LED
- added D3: LED_R, symbol Device:LED
- added FB1: FerriteBead, symbol Device:FerriteBead
- added J1: Conn_01x06, symbol Connector_Generic:Conn_01x06
- added J2: Conn_01x03, symbol Connector_Generic:Conn_01x03
- added J3: Conn_01x08, symbol Connector_Generic:Conn_01x08
- added R1, R2, R3: 0R, symbol Device:R
- added R10, R7, R9: R, symbol Device:R
- added R4, R5, R6: 1K, symbol Device:R
- added R8: 2K2, symbol Device:R
- added SW1: SW_DIP_x01, symbol Switch:SW_DIP_x01
- added TH1: 10K, symbol Device:Thermistor_NTC
- added U1: STM32F405RGTx, Package_QFP:LQFP-64_10x10mm_P0.5mm, symbol MCU_ST_STM32F4:STM32F405RGTx
- added Y1: Crystal, symbol Device:Crystal
Connections:
- new net: R1.2, U1.60 (BOOT0)
- new net: C11.1, C12.1, FB1.1, U1.13 (VDDA)
- new net: D3.2 (A), R6.2
- new net: C10.1, U1.47 (VCAP_2)
- new net: C9.1, U1.31 (VCAP_1)
- new net: R2.2, U1.5 (PH0)
- new net: R3.2, U1.6 (PH1)
- new net: C14.2, R2.1, Y1.2
- new net: C13.2, R3.1, Y1.1
- new net: D2.2 (A), R5.2
- new net: D1.2 (A), R4.2
- new net +3V3: C1.1, C16.1, C2.1, C3.1, C4.1, C5.1, C6.1, C7.1, FB1.2, J1.1 (Pin_1), J3.2 (Pin_2), R1.1, R4.1, TH1.1, U1.1 (VBAT), U1.19 (VDD), U1.32 (VDD), U1.48 (VDD), U1.64 (VDD)
- new net +5V: J2.1 (Pin_1), J2.3 (Pin_3), J3.1 (Pin_1), R7.2
- new net +VDC: R9.1
- new net ADC_TEMP: R8.1, TH1.2, U1.17 (PA3)
- new net AN_IN: C17.1, R10.1, R9.2, U1.10 (PC2)
- new net BR_SO1: U1.27 (PB1)
- new net BR_SO2: U1.26 (PB0)
- new net CAN_RX: U1.61 (PB8)
- new net CAN_TX: U1.62 (PB9)
- new net DC_CAL: U1.33 (PB12)
- new net EN_GATE: U1.51 (PC10)
- new net FAULT: U1.53 (PC12)
- new net GND: C1.2, C10.2, C11.2, C12.2, C13.1, C14.1, C15.2, C17.2, C2.2, C3.2, C4.2, C5.2, C6.2, C7.2, C8.2, C9.2, D1.1 (K), D2.1 (K), D3.1 (K), J1.3 (Pin_3), J2.2 (Pin_2), J3.3 (Pin_3), J3.8 (Pin_8), R10.2, R8.2, SW1.1, U1.12 (VSSA), U1.18 (VSS), U1.63 (VSS)
- new net H1: U1.43 (PA10)
- new net H2: U1.42 (PA9)
- new net H3: U1.41 (PA8)
- new net HALL2: U1.59 (PB7)
- new net HALL_1: U1.58 (PB6)
- new net HALL_3: U1.52 (PC11)
- new net L1: U1.36 (PB15)
- new net L2: U1.35 (PB14)
- new net L3: U1.34 (PB13)
- new net LED_GREEN: R5.1, U1.24 (PC4)
- new net LED_RED: R6.1, U1.25 (PC5)
- new net MISO_ADC_EXT2: J3.7 (Pin_7), U1.22 (PA6)
- new net NRST: C8.1, J1.5 (Pin_5), SW1.2, U1.7 (NRST)
- new net RX_SCL_MOSI: J3.6 (Pin_6), U1.23 (PA7), U1.29 (PB10), U1.38 (PC7)
- new net SCK_ADC_EXT: J3.4 (Pin_4), U1.21 (PA5)
- new net SENS1: U1.16 (PA2)
- new net SENS2: U1.15 (PA1)
- new net SENS3: U1.14 (PA0)
- new net SERVO: C15.1, R7.1, U1.57 (PB5)
- new net SWCLK: J1.2 (Pin_2), U1.49 (PA14)
- new net SWDIO: J1.4 (Pin_4), U1.46 (PA13)
- new net TEMP_MOTOR: U1.8 (PC0)
- new net TX_SDA_NSS: J3.5 (Pin_5), U1.20 (PA4), U1.30 (PB11), U1.37 (PC6)
- new net UDB_DP: U1.45 (PA12)
- new net USB_DN: U1.44 (PA11)
- no-connect marks 0 -> 13
Other:
- note added: "100nF Decoupling Capacitors place one as close as possible to each pin"
- note added: "Boost internally pulled up"
- note added: "COMMUNICATION"
- note added: "MCU"
- note added: "NTC_THERMISTOR"
- note added: "Programming/Debug"
- note added: "SERVO"
- note added: "VOLTAGE DIVIDER"
- note added: "WHEN VDC = 60V => AN_IN = 3V204"
- note added: "see boot modes Table 7"

Commit message: libraries & schemtics
Other:
- note added: "03407610395"
- note added: "Muhammad Moiz"
- note added: "moizrai765yt@gmail.com"
- company: (none) -> coVenture
- title: (none) -> MCU
Changed lines of the file:
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@@
 	(generator_version "8.0")
 	(paper "A4")
+	(title_block
+		(title "MCU")
+		(date "2025-02-03")
+		(rev "rev01_1")
+		(company "coVenture")
+	)
 	(junction
 		(at 264.16 121.92)
@@
 			(width 0)
 			(type default)
+		)
+	)
+	(text "Muhammad Moiz\n"
+		(exclude_from_sim no)
+		(at 210.566 168.656 0)
+		(effects
+			(font
+				(size 1.27 1.27)
+			)
 		)
 	)
@@
 		)
 	)
+	(text "03407610395\n"
+		(exclude_from_sim no)
+		(at 209.55 177.8 0)
+		(effects
+			(font
+				(size 1.27 1.27)
+			)
+		)
+	)
 	(text "WHEN VDC = 60V =>\nAN_IN = 3V204"
 		(exclude_from_sim no)
@@
 			)
 		)
+	)
+	(text "moizrai765yt@gmail.com\n"
+		(exclude_from_sim no)
+		(at 214.63 171.704 0)
+		(effects
+			(font
+				(size 1.27 1.27)
+			)
+		)

Commit message: updated footprints
Parts:
- removed C16: 100n, symbol Device:C
- removed C17: 10u, symbol Device:C
- removed R10, R9: R, symbol Device:R
- removed TH1: 10K, symbol Device:Thermistor_NTC
- added D13, D14, D16: BAT60A, Diode_SMD:D_SOD-323, symbol Diode:BAT60A
- added D15: SD05_SOD323, Diode_SMD:D_SOD-323, symbol Diode:SD05_SOD323
- C1, C10, C11, C12, C13, C14, C15, C2, C3, C4, C5, C6, C7, C8, C9: footprint (none) -> Capacitor_SMD:C_0603_1608Metric
- D1, D2, D3: footprint (none) -> LED_SMD:LED_1W_3W_R8
- FB1: footprint (none) -> Ferrite_THT:LairdTech_28C0236-0JW-10
- J1: footprint (none) -> Connector_PinHeader_1.00mm:PinHeader_1x06_P1.00mm_Vertical
- J2: footprint (none) -> Connector_PinHeader_1.00mm:PinHeader_1x03_P1.00mm_Vertical
- J3: footprint (none) -> Connector_PinHeader_1.00mm:PinHeader_1x08_P1.00mm_Vertical
- R1: value 0R -> 100R; footprint (none) -> Resistor_SMD:R_0201_0603Metric
- R2, R3, R4, R5, R6: footprint (none) -> Resistor_SMD:R_0201_0603Metric
- R7: value R -> 2k2; footprint (none) -> Resistor_SMD:R_0201_0603Metric
- R8: value 2K2 -> 2k2; footprint (none) -> Resistor_SMD:R_0201_0603Metric
- Y1: footprint (none) -> Crystal:Crystal_SMD_3215-2Pin_3.2x1.5mm
Connections:
- net +3V3: now also D13.1 (K), D14.1 (K); no longer J1.1 (Pin_1), J3.2 (Pin_2)
- net +5V: now also D16.1 (K); no longer J2.3 (Pin_3), J3.1 (Pin_1), R7.2
- net ADC_TEMP: no longer R8.1
- net GND: now also J1.5 (Pin_5), R8.1, D15.1 (A1); no longer R8.2, SW1.1
- net NRST: now also J1.6 (Pin_6); no longer J1.5 (Pin_5)
- net SWCLK: now also J1.4 (Pin_4); no longer J1.2 (Pin_2)
- net SWDIO: now also J1.2 (Pin_2); no longer J1.4 (Pin_4)
- net BOOT_P: now reaches R1.2, U1.60 (BOOT0)
- net +3V3_A: now reaches C11.1, C12.1, FB1.1, U1.13 (VDDA)
- net VCAP_2: now reaches C10.1, U1.47 (VCAP_2)
- net VCAP_1: now reaches C9.1, U1.31 (VCAP_1)
- net PH_0_P: now reaches R2.2, U1.5 (PH0)
- net PH_1_P: now reaches R3.2, U1.6 (PH1)
- net PH_0: now reaches C14.2, R2.1, Y1.2
- net PH_1: now reaches C13.2, R3.1, Y1.1
- new net: R8.2, SW1.1
- new net: J2.3 (Pin_3), R7.2
- new net +3V3_COM: D14.2 (A), J3.2 (Pin_2)
- new net +3V3_DBG: D13.2 (A), J1.1 (Pin_1)
- new net +5V_COM: D15.2 (A2), D16.2 (A), J3.1 (Pin_1)
- no-connect marks 13 -> 12
Other:
- note added: "FEEDBACK MCU"
- note added: "HALL ENCODER INPUT"
- note added: "NRST internally pulled up"
- note added: "OUTPUT PORTS"
- note added: "ROUTE AS DIFFERENTIAL PAIR"
- note added: "SENSING"
- note added: "USB"
- note removed: "Boost internally pulled up"
- note removed: "NTC_THERMISTOR"
- note removed: "VOLTAGE DIVIDER"
- note removed: "WHEN VDC = 60V => AN_IN = 3V204"
- moved on the sheet: FB1, R1

Commit message: UPDATED ERD ERRORS
Connections:
- net HALL2 is gone; now on net HALL_2_OUT: U1.59 (PB7)
- net HALL_1 is gone; now on net HALL_1_OUT: U1.58 (PB6)
- net HALL_3 is gone; now on net HALL_3_OUT: U1.52 (PC11)
- net UDB_DP is gone; now on net USB_P: U1.45 (PA12)
- net USB_DN is gone; now on net USB_N: U1.44 (PA11)
