File: Projects/Client Name/DF_ESC/Design/DF_ESC/DF_ESC_rev01_1/MOSFET DRIVER.kicad_sch (KiCad schematic)
At the start: 0 parts

Commit message: DRV8302
Parts:
- added C18: 120p, symbol Device:C
- added C19: 10n, symbol Device:C
- added C20, C21, C22, C23, C25: 2u2, symbol Device:C
- added C24: 22n, symbol Device:C
- added C26, C27, C28, C29, C30, C31, C32, C34, C35, C36: 10u, symbol Device:C
- added C33: 100u, symbol Device:C_Polarized_Small
- added C37, C38, C39: 220n, symbol Device:C
- added D4: PMEG6020AELR, Diode_SMD:Nexperia_CFP3_SOD-123W, symbol Diode:PMEG6020AELR
- added D5: BAT60A, Diode_SMD:D_SOD-323, symbol Diode:BAT60A
- added L1: 22u, symbol Device:L
- added R11: 205k, symbol Device:R
- added R12: 16k, symbol Device:R
- added R13: 10k, symbol Device:R
- added R14: 1M, symbol Device:R
- added R15: 18K, symbol Device:R
- added R16: 3K3, symbol Device:R
- added R17, R19, R21: 39k, symbol Device:R
- added R18, R20, R22: 2k2, symbol Device:R
- added U2: DRV8302DCAR, DCA56_6P35X3P61, symbol DRV8302:DRV8302DCAR
Connections:
- new net: C25.1, U2.27 (AVDD)
- new net: C19.1, R12.1
- new net +3V3: U2.24 (REF), U2.9 (M_OC)
- new net +5V: D5.1 (K)
- new net +5_DRV: C33.1, D5.2 (A), L1.2, R15.2
- new net +VDC: C26.1, C27.1, C28.1, C29.1, C30.1, C31.1, C34.2, C35.2, C36.2, U2.29 (PVDD1), U2.53 (PVDD2), U2.54 (PVDD2)
- new net BIAS: R14.1, U2.49 (BIAS)
- new net BR_SO1: U2.25 (SO1)
- new net BR_SO2: U2.26 (SO2)
- new net BST_A: C37.2, C38.2, C39.2, U2.48 (BST_A)
- new net BST_B: U2.43 (BST_B)
- new net BST_BK: C32.1, U2.52 (BST_BK)
- new net BST_C: U2.38 (BST_C)
- new net COMP: C18.2, R12.2, U2.2 (COMP)
- new net CP1: C24.1, U2.14 (CP1)
- new net CP2: C24.2, U2.15 (CP2)
- new net DC_CAL: U2.12 (DC_CAL)
- new net DTC: R13.2, U2.7 (DTC)
- new net DVDD: C20.1, C21.1, U2.11 (OC_ADJ), U2.23 (DVDD)
- new net EX_GATE: U2.16 (EN_GATE)
- new net FAULT: U2.6 (*FAULT)
- new net GND: C18.1, C19.2, C20.2, C21.2, C22.2, C23.2, C25.2, C26.2, C27.2, C28.2, C29.2, C30.2, C31.2, C33.2, C34.1, C35.1, C36.1, D4.2 (A), R11.1, R13.1, R14.2, R16.1, R18.1, R20.1, R22.1, U2.10 (GAIN), U2.28 (AGND), U2.57 (EPAD), U2.8 (M_PWM)
- new net GVDD: C22.1, C23.1, U2.13 (GVDD)
- new net H1: U2.17 (INH_A)
- new net H1_LOW: U2.44 (SL_A)
- new net H1_VS: C37.1, R21.2, U2.46 (SH_A)
- new net H2: U2.19 (INH_B)
- new net H2_LOW: U2.39 (SL_B)
- new net H2_VS: C38.1, R19.2, U2.41 (SH_B)
- new net H3: U2.21 (INH_C)
- new net H3_LOW: U2.34 (SL_C)
- new net H3_VS: C39.1, R17.2, U2.36 (SH_C)
- new net L1: U2.18 (INL_A)
- new net L2: U2.20 (INL_B)
- new net L3: U2.22 (INL_C)
- new net M_H1: U2.47 (GH_A)
- new net M_H2: U2.42 (GH_B)
- new net M_H3: U2.37 (GH_C)
- new net M_L1: U2.45 (GL_A)
- new net M_L2: U2.40 (GL_B)
- new net M_L3: U2.35 (GL_C)
- new net PH: C32.2, D4.1 (K), L1.1, U2.50 (PH), U2.51 (PH)
- new net RT_CLK: R11.2, U2.1 (RT_CLK)
- new net S1_N: U2.30 (SP2), U2.31 (SN2), U2.32 (SP1), U2.33 (SN1)
- new net SENS1: R17.1, R18.2
- new net SENS2: R19.1, R20.2
- new net SENS3: R21.1, R22.2
- new net VSENSE: R15.1, R16.2, U2.3 (VSENSE)
- no-connect marks 0 -> 4
Other:
- note added: "10u DECOUPING CAPs KEEP AS CLOSE AS POSSIBLE TO THE IC"
- note added: "BOOTSTRAP CAPs"
- note added: "BULK CAPACITANCE KEEP AS CLOSE TO THE IC AND TO THE DRIVER INPUT LOOP"
- note added: "Hx_Vx"
- note added: "INPUT PORTS"
- note added: "KEEP AWAY FROM NOISY TRACKS AND COMPONENTS"
- note added: "MCU SENSING FEEDBACK FOR EACH PHASE"
- note added: "MOSFET DRIVER"
- note added: "OUTPUT PORTS"
- note added: "PHASE 1"
- note added: "PHASE 2"
- note added: "PHASE 3"
- note added: "SENSE 1 - PHASE 1"
- note added: "SENSE 2 - PHASE 2"
- company: (none) -> coVenture
- title: (none) -> MOSFET DRIVER

Commit message: libraries & schemtics
Other:
- note added: "03407610395"
- note added: "Muhammad Moiz"
- note added: "moizrai765yt@gmail.com"
Changed lines of the file:
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@@
 	(title_block
 		(title "MOSFET DRIVER")
-		(date "2025-01-30")
+		(date "2025-02-03")
+		(rev "rev01_1")
 		(company "coVenture")
 	)
@@
 		)
 	)
+	(text "03407610395\n"
+		(exclude_from_sim no)
+		(at 209.55 177.8 0)
+		(effects
+			(font
+				(size 1.27 1.27)
+			)
+		)
+	)
 	(text "OUTPUT PORTS"
 		(exclude_from_sim no)
@@
 			)
 		)
+	)
+	(text "moizrai765yt@gmail.com\n"
+		(exclude_from_sim no)
+		(at 214.63 171.704 0)
+		(effects
+			(font
+				(size 1.27 1.27)
+			)
+		)
+	)
+	(text "Muhammad Moiz\n"
+		(exclude_from_sim no)
+		(at 210.566 168.656 0)
+		(effects
+			(font
+				(size 1.27 1.27)
+			)
+		)

Commit message: updated footprints
Parts:
- C18, C19, C20, C21, C22, C23, C24, C25, C26, C27, C28, C29, C30, C31, C32, C33, C34, C35, C36, C37, C38, C39: footprint (none) -> Capacitor_SMD:C_0603_1608Metric
- L1: footprint (none) -> Inductor_SMD:L_0201_0603Metric
- R11, R12, R13, R14, R15, R16, R17, R18, R19, R20, R21, R22: footprint (none) -> Resistor_SMD:R_0201_0603Metric
- U2: footprint DCA56_6P35X3P61 -> DRV8302DCAR:DCA56_6P35X3P61
Changed lines of the file:
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@@
 			)
 		)
-		(property "Footprint" ""
+		(property "Footprint" "Resistor_SMD:R_0201_0603Metric"
 			(at 277.368 134.62 90)
 			(effects
@@
 			)
 		)
-		(property "Footprint" ""
+		(property "Footprint" "Resistor_SMD:R_0201_0603Metric"
 			(at 241.808 134.62 90)
 			(effects
@@
 			)
 		)
-		(property "Footprint" ""
+		(property "Footprint" "Capacitor_SMD:C_0603_1608Metric"
 			(at 204.47 76.2 0)
 			(effects
@@
 			)
 		)
-		(property "Footprint" ""
+		(property "Footprint" "Capacitor_SMD:C_0603_1608Metric"
 			(at 178.7652 50.8 0)
 			(effects
@@
 			)
 		)
-		(property "Footprint" ""
+		(property "Footprint" "Capacitor_SMD:C_0603_1608Metric"
 			(at 67.0052 57.15 0)
 			(effects
@@
 			)
 		)
-		(property "Footprint" ""
+		(property "Footprint" "Capacitor_SMD:C_0603_1608Metric"
 			(at 194.0052 50.8 0)
 			(effects
@@
 			)
 		)
-		(property "Footprint" ""
+		(property "Footprint" "Resistor_SMD:R_0201_0603Metric"
 			(at 259.588 134.62 90)
 			(effects
@@
 			)
 		)
-		(property "Footprint" ""
+		(property "Footprint" "Resistor_SMD:R_0201_0603Metric"
 			(at 218.948 76.2 90)
 			(effects
@@
 			)
 		)
-		(property "Footprint" ""
+		(property "Footprint" "Capacitor_SMD:C_0603_1608Metric"
 			(at 73.3552 101.6 0)
 			(effects
@@
 			)
 		)
-		(property "Footprint" ""
+		(property "Footprint" "Capacitor_SMD:C_0603_1608Metric"
 			(at 199.6948 139.7 0)
 			(effects
@@
 			)
 		)
-		(property "Footprint" ""
+		(property "Footprint" "Resistor_SMD:R_0201_0603Metric"
 			(at 157.48 80.518 90)
 			(effects
@@
 			)
 		)
-		(property "Footprint" "DCA56_6P35X3P61"
+		(property "Footprint" "DRV8302DCAR:DCA56_6P35X3P61"
 			(at 96.52 60.96 0)
 			(effects
@@
 			)
 		)
-		(property "Footprint" ""
+		(property "Footprint" "Capacitor_SMD:C_0603_1608Metric"
 			(at 168.6052 50.8 0)
 			(effects
@@
 			)
 		)
-		(property "Footprint" ""
+		(property "Footprint" "Resistor_SMD:R_0201_0603Metric"
 			(at 83.82 77.978 90)
 			(effects
@@
 			)
 		)
-		(property "Footprint" ""
+		(property "Footprint" "Capacitor_SMD:C_0603_1608Metric"
 			(at 183.8452 50.8 0)
 			(effects
@@
 			)
 		)
-		(property "Footprint" ""
+		(property "Footprint" "Capacitor_SMD:C_0603_1608Metric"
 			(at 189.5348 139.7 0)
 			(effects
@@
 			)
 		)
-		(property "Footprint" ""
+		(property "Footprint" "Capacitor_SMD:C_0603_1608Metric"
 			(at 160.3248 135.89 0)
 			(effects
@@
 			)
 		)
-		(property "Footprint" ""
+		(property "Footprint" "Capacitor_SMD:C_0603_1608Metric"
 			(at 173.6852 50.8 0)
 			(effects
@@
 			)
 		)
-		(property "Footprint" ""
+		(property "Footprint" "Capacitor_SMD:C_0603_1608Metric"
 			(at 50.4952 114.3 0)
 			(effects
@@
 			)
 		)
-		(property "Footprint" ""
+		(property "Footprint" "Capacitor_SMD:C_0603_1608Metric"
 			(at 209.8548 139.7 0)
 			(effects
@@
 			)
 		)
-		(property "Footprint" ""
+		(property "Footprint" "Capacitor_SMD:C_0603_1608Metric"
 			(at 188.9252 50.8 0)
 			(effects
@@
 			)
 		)
-		(property "Footprint" ""
+		(property "Footprint" "Resistor_SMD:R_0201_0603Metric"
 			(at 55.372 58.42 90)
 			(effects
@@
 			)
 		)
-		(property "Footprint" ""
+		(property "Footprint" "Capacitor_SMD:C_0603_1608Metric"
 			(at 162.56 70.1548 0)
 			(effects
@@
 			)
 		)
-		(property "Footprint" ""
+		(property "Footprint" "Capacitor_SMD:C_0603_1608Metric"
 			(at 50.4952 99.06 0)
 			(effects
@@
 			)
 		)
-		(property "Footprint" ""
+		(property "Footprint" "Resistor_SMD:R_0201_0603Metric"
 			(at 259.588 144.78 90)
 			(effects
@@
 			)
 		)
-		(property "Footprint" ""
+		(property "Footprint" "Capacitor_SMD:C_0603_1608Metric"
 			(at 60.6552 99.06 0)
 			(effects
@@
 			)
 		)
-		(property "Footprint" ""
+		(property "Footprint" "Inductor_SMD:L_0201_0603Metric"
 			(at 186.69 71.12 0)
 			(effects
@@
 			)
 		)
-		(property "Footprint" ""
+		(property "Footprint" "Capacitor_SMD:C_0603_1608Metric"
 			(at 142.5448 135.89 0)
 			(effects
@@
 			)
 		)
-		(property "Footprint" ""
+		(property "Footprint" "Capacitor_SMD:C_0603_1608Metric"
 			(at 60.6552 114.3 0)
 			(effects
@@
 			)
 		)
-		(property "Footprint" ""
+		(property "Footprint" "Capacitor_SMD:C_0603_1608Metric"
 			(at 56.1848 44.45 0)
 			(effects
@@
 			)
 		)
-		(property "Footprint" ""
+		(property "Footprint" "Capacitor_SMD:C_0603_1608Metric"
 			(at 83.5152 135.89 0)
 			(effects
@@
 			)
 		)
-		(property "Footprint" ""
+		(property "Footprint" "Resistor_SMD:R_0201_0603Metric"
 			(at 241.808 144.78 90)
 			(effects
@@
 			)
 		)
-		(property "Footprint" ""
+		(property "Footprint" "Resistor_SMD:R_0201_0603Metric"
 			(at 218.948 86.36 90)
 			(effects
@@
 			)
 		)
-		(property "Footprint" ""
+		(property "Footprint" "Resistor_SMD:R_0201_0603Metric"
 			(at 277.368 144.78 90)
 			(effects
@@
 			)
 		)
-		(property "Footprint" ""
+		(property "Footprint" "Capacitor_SMD:C_0603_1608Metric"
 			(at 151.4348 135.89 0)
 			(effects
@@
 			)
 		)
-		(property "Footprint" ""
+		(property "Footprint" "Resistor_SMD:R_0201_0603Metric"
 			(at 76.962 53.34 90)
 			(effects

Commit message: UPDATED ERD ERRORS
Parts:
- removed C33: 100u, Capacitor_SMD:C_0603_1608Metric, symbol Device:C_Polarized_Small
- added C16, C17, C33: 10u, Capacitor_SMD:C_0603_1608Metric, symbol Device:C
- added NT9: NetTie_2, symbol Device:NetTie_2
Connections:
- net +5_DRV: now also C16.2, C17.2, C33.2
- net BST_A: no longer C38.2, C39.2
- net BST_B: now also C38.2
- net BST_C: now also C39.2
- net DVDD: now also NT9.1; no longer C20.1, C21.1, U2.11 (OC_ADJ)
- net GND: now also C16.1, C17.1, C33.1
- net EX_GATE renamed EN_GATE
- new net OC_ADJ: C20.1, C21.1, NT9.2, U2.11 (OC_ADJ)
