File: Projects/Client Name/DF_ESC/Design/DF_ESC/DF_ESC_rev01_1/STEP-DOWN.kicad_sch (KiCad schematic)
At the start: 10 parts, among them U4 AMS1117-3.3

Commit message: updated footprints
Parts:
- C51, C52, C53, C54: footprint (none) -> Capacitor_SMD:C_0603_1608Metric
- D7, D9: footprint (none) -> LED_SMD:LED_1W_3W_R8
- R35, R36: footprint (none) -> Resistor_SMD:R_0201_0603Metric
Changed lines of the file:
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@@
 			)
 		)
-		(property "Footprint" ""
+		(property "Footprint" "Capacitor_SMD:C_0603_1608Metric"
 			(at 147.0152 74.93 0)
 			(effects
@@
 			)
 		)
-		(property "Footprint" ""
+		(property "Footprint" "Resistor_SMD:R_0201_0603Metric"
 			(at 62.992 71.12 90)
 			(effects
@@
 			)
 		)
-		(property "Footprint" ""
+		(property "Footprint" "Capacitor_SMD:C_0603_1608Metric"
 			(at 135.5852 74.93 0)
 			(effects
@@
 			)
 		)
-		(property "Footprint" ""
+		(property "Footprint" "LED_SMD:LED_1W_3W_R8"
 			(at 190.5 86.36 0)
 			(effects
@@
 			)
 		)
-		(property "Footprint" ""
+		(property "Footprint" "Capacitor_SMD:C_0603_1608Metric"
 			(at 80.9752 74.93 0)
 			(effects
@@
 			)
 		)
-		(property "Footprint" ""
+		(property "Footprint" "Capacitor_SMD:C_0603_1608Metric"
 			(at 92.4052 74.93 0)
 			(effects
@@
 			)
 		)
-		(property "Footprint" ""
+		(property "Footprint" "LED_SMD:LED_1W_3W_R8"
 			(at 64.77 86.36 0)
 			(effects
@@
 			)
 		)
-		(property "Footprint" ""
+		(property "Footprint" "Resistor_SMD:R_0201_0603Metric"
 			(at 188.722 71.12 90)
 			(effects

Commit message: UPDATED ERD ERRORS
Changed lines of the file:
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@@
+	)
+	(junction
+		(at 140.97 77.47)
+		(diameter 0)
+		(color 0 0 0 0)
 	)
 	(junction
@@
 	)
 	(junction
-		(at 140.97 74.93)
-		(diameter 0)
-		(color 0 0 0 0)
-	)
-	(junction
 		(at 134.62 67.31)
 		(diameter 0)
@@
 	(wire
 		(pts
+			(xy 146.05 77.47) (xy 146.05 74.93)
+		)
+		(stroke
+			(width 0)
+			(type default)
+		)
+	)
+	(wire
+		(pts
 			(xy 146.05 67.31) (xy 171.45 67.31)
 		)
@@
 		)
 	)
+	(wire
+		(pts
+			(xy 134.62 77.47) (xy 134.62 74.93)
+		)
+		(stroke
+			(width 0)
+			(type default)
+		)
+	)
 	(polyline
 		(pts
@@
 	(wire
 		(pts
-			(xy 134.62 74.93) (xy 140.97 74.93)
+			(xy 134.62 77.47) (xy 140.97 77.47)
 		)
 		(stroke
@@
 	(wire
 		(pts
-			(xy 140.97 74.93) (xy 146.05 74.93)
+			(xy 140.97 77.47) (xy 146.05 77.47)
 		)
 		(stroke
@@
 	(symbol
 		(lib_id "power:GND")
-		(at 140.97 74.93 0)
+		(at 140.97 77.47 0)
 		(unit 1)
 		(exclude_from_sim no)
@@
 		(fields_autoplaced yes)
 		(property "Reference" "#PWR073"
-			(at 140.97 81.28 0)
+			(at 140.97 83.82 0)
 			(effects
 				(font
@@
 		)
 		(property "Value" "GND"
-			(at 140.97 80.01 0)
+			(at 140.97 82.55 0)
 			(effects
 				(font
@@
 		)
 		(property "Footprint" ""
-			(at 140.97 74.93 0)
+			(at 140.97 77.47 0)
 			(effects
 				(font
@@
 		)
 		(property "Datasheet" ""
-			(at 140.97 74.93 0)
+			(at 140.97 77.47 0)
 			(effects
 				(font
@@
 		)
 		(property "Description" "Power symbol creates a global label with name \"GND\" , ground"
-			(at 140.97 74.93 0)
-			(effects
-				(font
+			(at 140.97 77.47 0)
+			(effects
+				(font
