File: Projects/Client Name/DF_ESC/Design/DF_ESC/DF_ESC_rev01_1/USB.kicad_sch (KiCad schematic)
At the start: 9 parts, among them J6 USB_C_Receptacle_USB2.0_16P

Commit message: updated footprints
Parts:
- D10: footprint PUSB3AB6Z -> PUSB3A6Z:PUSB3AB6Z
- J6: footprint (none) -> Connector_USB:USB_C_Plug_Molex_105444
- R37, R38, R39, R40, R41, R42, R43: footprint (none) -> Resistor_SMD:R_0201_0603Metric
Changed lines of the file:
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@@
 	)
 	(global_label "USB_N"
-		(shape input)
+		(shape bidirectional)
 		(at 267.97 54.61 0)
 		(fields_autoplaced yes)
@@
 		)
 		(property "Intersheetrefs" "${INTERSHEET_REFS}"
-			(at 277.1584 54.61 0)
+			(at 278.1744 54.61 0)
 			(effects
 				(font
@@
 	)
 	(global_label "USB_P"
-		(shape input)
+		(shape bidirectional)
 		(at 267.97 58.42 0)
 		(fields_autoplaced yes)
@@
 		)
 		(property "Intersheetrefs" "${INTERSHEET_REFS}"
-			(at 277.0979 58.42 0)
+			(at 278.1139 58.42 0)
 			(effects
 				(font
@@
 			)
 		)
-		(property "Footprint" ""
+		(property "Footprint" "Connector_USB:USB_C_Plug_Molex_105444"
 			(at 60.96 73.66 0)
 			(effects
@@
 			)
 		)
-		(property "Footprint" ""
+		(property "Footprint" "Resistor_SMD:R_0201_0603Metric"
 			(at 193.04 50.038 90)
 			(effects
@@
 			)
 		)
-		(property "Footprint" ""
+		(property "Footprint" "Resistor_SMD:R_0201_0603Metric"
 			(at 47.752 102.87 90)
 			(effects
@@
 			)
 		)
-		(property "Footprint" ""
+		(property "Footprint" "Resistor_SMD:R_0201_0603Metric"
 			(at 43.942 102.87 90)
 			(effects
@@
 			)
 		)
-		(property "Footprint" ""
+		(property "Footprint" "Resistor_SMD:R_0201_0603Metric"
 			(at 193.04 55.118 90)
 			(effects
@@
 			)
 		)
-		(property "Footprint" ""
+		(property "Footprint" "Resistor_SMD:R_0201_0603Metric"
 			(at 123.952 67.31 90)
 			(effects
@@
 			)
 		)
-		(property "Footprint" ""
+		(property "Footprint" "Resistor_SMD:R_0201_0603Metric"
 			(at 113.792 69.85 90)
 			(effects
@@
 			)
 		)
-		(property "Footprint" "PUSB3AB6Z"
+		(property "Footprint" "PUSB3A6Z:PUSB3AB6Z"
 			(at 201.93 187.63 0)
 			(effects
@@
 			)
 		)
-		(property "Footprint" ""
+		(property "Footprint" "Resistor_SMD:R_0201_0603Metric"
 			(at 85.852 45.72 90)
 			(effects

Commit message: UPDATED ERD ERRORS
Connections:
- net USB-C_N: now also D10.6 (CH5), J6.A7 (D-), J6.B7 (D-), R42.1
- net USB-C_P: now also D10.7 (CH6), J6.A6 (D+), J6.B6 (D+), R43.1
- net USB_N: now also R42.2
- net USB_P: now also R43.2
